File: Hardware/TrainingBoard2020.sch (KiCad schematic (older format))
At the start: 0 parts

Commit message: Created Training Board
Changed lines of the file:
@@
 $EndDescr
 $Sheet
-S 1725 1925 1800 1600
+S 4400 3175 1825 1600
+U 5F4E3D8B
+F0 "Buttons" 50
+F1 "TrainingBoard02.sch" 50
+$EndSheet
+$Sheet
+S 6550 3175 1875 1600
+U 5F5029F1
+F0 "Connectors" 50
+F1 "TrainingBoard03.sch" 50
+$EndSheet
+$Sheet
+S 2225 3175 1800 1600
 U 5F525D93
 F0 "Power" 50
 F1 "TrainingBoard01.sch" 50
 $EndSheet
-Text HLabel 3525 3175 0    50   Output ~ 0
-+3.3V
-$Sheet
-S 3900 1925 1825 1600
-U 5F4E3D8B
-F0 "Buttons" 50
-F1 "TrainingBoard02.sch" 50
-$EndSheet
-Text HLabel 3900 3175 2    50   Input ~ 0
-+3.3V
-$Sheet
-S 6150 1875 2025 1675
-U 5F5029F1
-F0 "Connectors" 50
-F1 "TrainingBoard03.sch" 50
-$EndSheet
-Wire Wire Line
-	3525 3175 3900 3175
 $EndSCHEMATC
