File: Hardware/TrainingBoard02.sch (KiCad schematic (older format))
At the start: 15 parts

Commit message: made board
Parts:
- removed R? (x2): 1k, symbol Device:R
- removed SW? (x2): SW_Push, symbol Switch:SW_Push
- added R? (x2): 1k, symbol Device:R
- added SW? (x2): SW_Push, symbol Switch:SW_Push
Connections:
- net GND: now also SW?.1, SW?.1
- net IND_1: now also R?.1, SW?.2; no longer C?.1, R?.2
- net IND_2: now also R?.1, SW?.2; no longer C?.1, R?.2, R?.2
- net IND_3: now also R?.1, SW?.2; no longer C?.1, R?.2
- new net: C?.1, R?.2, R?.2 (x3)
Other:
- moved on the sheet: C?, SW?
Changed lines of the file:
@@
 $Descr A4 11693 8268
 encoding utf-8
-Sheet 3 4
+Sheet 2 4
 Title ""
 Date ""
@@
 $EndComp
 $Comp
-L Switch:SW_Push SW?
-U 1 1 5F5657AD
-P 3025 4100
-F 0 "SW?" H 3025 4385 50  0000 C CNN
-F 1 "SW_Push" H 3025 4294 50  0000 C CNN
-F 2 "" H 3025 4300 50  0001 C CNN
-F 3 "~" H 3025 4300 50  0001 C CNN
-	1    3025 4100
-	1    0    0    -1
-$EndComp
-$Comp
 L Device:R R?
 U 1 1 5F566AF5
@@
 L Device:C C?
 U 1 1 5F566E39
-P 3850 4400
-F 0 "C?" H 3965 4446 50  0000 L CNN
-F 1 "0.1uF" H 3965 4355 50  0000 L CNN
-F 2 "" H 3888 4250 50  0001 C CNN
-F 3 "~" H 3850 4400 50  0001 C CNN
-	1    3850 4400
-	1    0    0    -1
-$EndComp
-$Comp
-L power:GND #PWR?
-U 1 1 5F567207
-P 2700 4200
-F 0 "#PWR?" H 2700 3950 50  0001 C CNN
-F 1 "GND" H 2705 4027 50  0000 C CNN
-F 2 "" H 2700 4200 50  0001 C CNN
-F 3 "" H 2700 4200 50  0001 C CNN
-	1    2700 4200
+P 3975 4400
+F 0 "C?" H 4090 4446 50  0000 L CNN
+F 1 "0.1uF" H 4090 4355 50  0000 L CNN
+F 2 "" H 4013 4250 50  0001 C CNN
+F 3 "~" H 3975 4400 50  0001 C CNN
+	1    3975 4400
 	1    0    0    -1
 $EndComp
@@
 $EndComp
 $Comp
-L Device:R R?
-U 1 1 5F568B38
-P 3550 4100
-F 0 "R?" V 3725 4050 50  0000 L CNN
-F 1 "1k" V 3650 4075 50  0000 L CNN
-F 2 "" V 3480 4100 50  0001 C CNN
-F 3 "~" H 3550 4100 50  0001 C CNN
-	1    3550 4100
-	0    -1   -1   0
-$EndComp
-$Comp
 L power:GND #PWR?
 U 1 1 5F56A4E8
-P 3850 4650
-F 0 "#PWR?" H 3850 4400 50  0001 C CNN
-F 1 "GND" H 3855 4477 50  0000 C CNN
-F 2 "" H 3850 4650 50  0001 C CNN
-F 3 "" H 3850 4650 50  0001 C CNN
-	1    3850 4650
-	1    0    0    -1
-$EndComp
-Wire Wire Line
-	2700 4200 2700 4100
-Wire Wire Line
-	2700 4100 2825 4100
-Wire Wire Line
-	3225 4100 3400 4100
+P 3975 4650
+F 0 "#PWR?" H 3975 4400 50  0001 C CNN
+F 1 "GND" H 3980 4477 50  0000 C CNN
+F 2 "" H 3975 4650 50  0001 C CNN
+F 3 "" H 3975 4650 50  0001 C CNN
+	1    3975 4650
+	1    0    0    -1
+$EndComp
 Wire Wire Line
 	3975 4100 3975 3850
 Wire Wire Line
-	3850 4250 3850 4100
-Wire Wire Line
-	3700 4100 3850 4100
-Connection ~ 3850 4100
-Wire Wire Line
-	3850 4100 3975 4100
-Wire Wire Line
-	3850 4550 3850 4650
-Wire Wire Line
-	3975 4100 4100 4100
-Connection ~ 3975 4100
+	3975 4250 3975 4100
+Wire Wire Line
+	3975 4550 3975 4650
 Wire Wire Line
 	3975 3550 3975 3425
 Wire Wire Line
 	3975 3125 3975 3000
-Text GLabel 4100 4100 2    50   Output ~ 0
-IND_1
 Text Notes 4100 3450 0    50   ~ 0
 Yellow
@@
 L Switch:SW_Push SW?
 U 1 1 5F56DB9F
-P 5125 4100
-F 0 "SW?" H 5125 4385 50  0000 C CNN
-F 1 "SW_Push" H 5125 4294 50  0000 C CNN
-F 2 "" H 5125 4300 50  0001 C CNN
-F 3 "~" H 5125 4300 50  0001 C CNN
-	1    5125 4100
+P 5100 4100
+F 0 "SW?" H 5100 4385 50  0000 C CNN
+F 1 "SW_Push" H 5100 4294 50  0000 C CNN
+F 2 "" H 5100 4300 50  0001 C CNN
+F 3 "~" H 5100 4300 50  0001 C CNN
+	1    5100 4100
 	1    0    0    -1
 $EndComp
@@
 L Device:C C?
 U 1 1 5F56DBAB
-P 5950 4400
-F 0 "C?" H 6065 4446 50  0000 L CNN
-F 1 "0.1uF" H 6065 4355 50  0000 L CNN
-F 2 "" H 5988 4250 50  0001 C CNN
-F 3 "~" H 5950 4400 50  0001 C CNN
-	1    5950 4400
+P 6075 4400
+F 0 "C?" H 6190 4446 50  0000 L CNN
+F 1 "0.1uF" H 6190 4355 50  0000 L CNN
+F 2 "" H 6113 4250 50  0001 C CNN
+F 3 "~" H 6075 4400 50  0001 C CNN
+	1    6075 4400
 	1    0    0    -1
 $EndComp
@@
 $EndComp
 $Comp
-L Device:R R?
-U 1 1 5F56DBBD
-P 5650 4100
-F 0 "R?" V 5825 4050 50  0000 L CNN
-F 1 "1k" V 5750 4075 50  0000 L CNN
-F 2 "" V 5580 4100 50  0001 C CNN
-F 3 "~" H 5650 4100 50  0001 C CNN
-	1    5650 4100
-	0    -1   -1   0
-$EndComp
-$Comp
 L power:GND #PWR?
 U 1 1 5F56DBC3
-P 5950 4650
-F 0 "#PWR?" H 5950 4400 50  0001 C CNN
-F 1 "GND" H 5955 4477 50  0000 C CNN
-F 2 "" H 5950 4650 50  0001 C CNN
-F 3 "" H 5950 4650 50  0001 C CNN
-	1    5950 4650
+P 6075 4650
+F 0 "#PWR?" H 6075 4400 50  0001 C CNN
+F 1 "GND" H 6080 4477 50  0000 C CNN
+F 2 "" H 6075 4650 50  0001 C CNN
+F 3 "" H 6075 4650 50  0001 C CNN
+	1    6075 4650
 	1    0    0    -1
 $EndComp
@@
 	4800 4200 4800 4100
 Wire Wire Line
-	4800 4100 4925 4100
-Wire Wire Line
-	5325 4100 5500 4100
-Wire Wire Line
-	6075 4100 6075 3850
-Wire Wire Line
-	5950 4250 5950 4100
-Wire Wire Line
-	5800 4100 5950 4100
-Connection ~ 5950 4100
-Wire Wire Line
-	5950 4100 6075 4100
-Wire Wire Line
-	5950 4550 5950 4650
-Wire Wire Line
-	6075 4100 6200 4100
-Connection ~ 6075 4100
+	6075 4550 6075 4650
 Wire Wire Line
 	6075 3550 6075 3425
 Wire Wire Line
 	6075 3125 6075 3000
-Text GLabel 6200 4100 2    50   Output ~ 0
+Text GLabel 5500 4350 2    50   Output ~ 0
 IND_2
 Text Notes 6200 3450 0    50   ~ 0
@@
 $EndComp
 $Comp
-L Switch:SW_Push SW?
-U 1 1 5F5739F7
-P 7225 4100
-F 0 "SW?" H 7225 4385 50  0000 C CNN
-F 1 "SW_Push" H 7225 4294 50  0000 C CNN
-F 2 "" H 7225 4300 50  0001 C CNN
-F 3 "~" H 7225 4300 50  0001 C CNN
-	1    7225 4100
-	1    0    0    -1
-$EndComp
-$Comp
 L Device:R R?
 U 1 1 5F5739FD
@@
 L Device:C C?
 U 1 1 5F573A03
-P 8050 4400
-F 0 "C?" H 8165 4446 50  0000 L CNN
-F 1 "0.1uF" H 8165 4355 50  0000 L CNN
-F 2 "" H 8088 4250 50  0001 C CNN
-F 3 "~" H 8050 4400 50  0001 C CNN
-	1    8050 4400
-	1    0    0    -1
-$EndComp
-$Comp
-L power:GND #PWR?
-U 1 1 5F573A09
-P 6900 4200
-F 0 "#PWR?" H 6900 3950 50  0001 C CNN
-F 1 "GND" H 6905 4027 50  0000 C CNN
-F 2 "" H 6900 4200 50  0001 C CNN
-F 3 "" H 6900 4200 50  0001 C CNN
-	1    6900 4200
+P 8175 4400
+F 0 "C?" H 8290 4446 50  0000 L CNN
+F 1 "0.1uF" H 8290 4355 50  0000 L CNN
+F 2 "" H 8213 4250 50  0001 C CNN
+F 3 "~" H 8175 4400 50  0001 C CNN
+	1    8175 4400
 	1    0    0    -1
 $EndComp
@@
 $EndComp
 $Comp
-L Device:R R?
-U 1 1 5F573A15
+L power:GND #PWR?
+U 1 1 5F573A1B
+P 8175 4650
+F 0 "#PWR?" H 8175 4400 50  0001 C CNN
+F 1 "GND" H 8180 4477 50  0000 C CNN
+F 2 "" H 8175 4650 50  0001 C CNN
+F 3 "" H 8175 4650 50  0001 C CNN
+	1    8175 4650
+	1    0    0    -1
+$EndComp
+Wire Wire Line
+	8175 4100 8175 3850
+Wire Wire Line
+	8175 4250 8175 4100
+Wire Wire Line
+	8175 4550 8175 4650
+Wire Wire Line
+	8175 3550 8175 3425
+Wire Wire Line
+	8175 3125 8175 3000
+Text Notes 8300 3450 0    50   ~ 0
+Yellow
+Connection ~ 6075 4100
+Wire Wire Line
+	6075 4250 6075 4100
+Wire Wire Line
+	6075 4100 6075 3850
+Wire Wire Line
+	5800 4100 6075 4100
+$Comp
+L Device:R R?
+U 1 1 5F56DBBD
+P 5650 4100
+F 0 "R?" V 5825 4050 50  0000 L CNN
+F 1 "1k" V 5750 4075 50  0000 L CNN
+F 2 "" V 5580 4100 50  0001 C CNN
+F 3 "~" H 5650 4100 50  0001 C CNN
+	1    5650 4100
+	0    -1   -1   0
+$EndComp
+Connection ~ 5400 4100
+Wire Wire Line
+	5400 4100 5500 4100
+Wire Wire Line
+	5400 4350 5500 4350
+Wire Wire Line
+	5400 4100 5400 4350
+Wire Wire Line
+	5300 4100 5400 4100
+Wire Wire Line
+	4900 4100 4800 4100
+Wire Wire Line
+	2800 4100 2700 4100
+Wire Wire Line
+	3200 4100 3300 4100
+Wire Wire Line
+	3300 4100 3300 4350
+Wire Wire Line
+	3300 4350 3400 4350
+Wire Wire Line
+	3300 4100 3400 4100
+Connection ~ 3300 4100
+$Comp
+L Device:R R?
+U 1 1 5F58E0DD
+P 3550 4100
+F 0 "R?" V 3725 4050 50  0000 L CNN
+F 1 "1k" V 3650 4075 50  0000 L CNN
+F 2 "" V 3480 4100 50  0001 C CNN
+F 3 "~" H 3550 4100 50  0001 C CNN
+	1    3550 4100
+	0    -1   -1   0
+$EndComp
+Text GLabel 3400 4350 2    50   Output ~ 0
+IND_1
+Wire Wire Line
+	2700 4200 2700 4100
+$Comp
+L power:GND #PWR?
+U 1 1 5F58E0D5
+P 2700 4200
+F 0 "#PWR?" H 2700 3950 50  0001 C CNN
+F 1 "GND" H 2705 4027 50  0000 C CNN
+F 2 "" H 2700 4200 50  0001 C CNN
+F 3 "" H 2700 4200 50  0001 C CNN
+	1    2700 4200
+	1    0    0    -1
+$EndComp
+$Comp
+L Switch:SW_Push SW?
+U 1 1 5F58E0CF
+P 3000 4100
+F 0 "SW?" H 3000 4385 50  0000 C CNN
+F 1 "SW_Push" H 3000 4294 50  0000 C CNN
+F 2 "" H 3000 4300 50  0001 C CNN
+F 3 "~" H 3000 4300 50  0001 C CNN
+	1    3000 4100
+	1    0    0    -1
+$EndComp
+Connection ~ 3975 4100
+Wire Wire Line
+	3700 4100 3975 4100
+$Comp
+L Switch:SW_Push SW?
+U 1 1 5F595C41
+P 7200 4100
+F 0 "SW?" H 7200 4385 50  0000 C CNN
+F 1 "SW_Push" H 7200 4294 50  0000 C CNN
+F 2 "" H 7200 4300 50  0001 C CNN
+F 3 "~" H 7200 4300 50  0001 C CNN
+	1    7200 4100
+	1    0    0    -1
+$EndComp
+$Comp
+L power:GND #PWR?
+U 1 1 5F595C47
+P 6900 4200
+F 0 "#PWR?" H 6900 3950 50  0001 C CNN
+F 1 "GND" H 6905 4027 50  0000 C CNN
+F 2 "" H 6900 4200 50  0001 C CNN
+F 3 "" H 6900 4200 50  0001 C CNN
+	1    6900 4200
+	1    0    0    -1
+$EndComp
+Wire Wire Line
+	6900 4200 6900 4100
+Text GLabel 7600 4350 2    50   Output ~ 0
+IND_3
+$Comp
+L Device:R R?
+U 1 1 5F595C4F
 P 7750 4100
 F 0 "R?" V 7925 4050 50  0000 L CNN
@@
 	0    -1   -1   0
 $EndComp
-$Comp
-L power:GND #PWR?
-U 1 1 5F573A1B
-P 8050 4650
-F 0 "#PWR?" H 8050 4400 50  0001 C CNN
-F 1 "GND" H 8055 4477 50  0000 C CNN
-F 2 "" H 8050 4650 50  0001 C CNN
-F 3 "" H 8050 4650 50  0001 C CNN
-	1    8050 4650
-	1    0    0    -1
-$EndComp
-Wire Wire Line
-	6900 4200 6900 4100
-Wire Wire Line
-	6900 4100 7025 4100
-Wire Wire Line
-	7425 4100 7600 4100
-Wire Wire Line
-	8175 4100 8175 3850
-Wire Wire Line
-	8050 4250 8050 4100
-Wire Wire Line
-	7900 4100 8050 4100
-Connection ~ 8050 4100
-Wire Wire Line
-	8050 4100 8175 4100
-Wire Wire Line
-	8050 4550 8050 4650
-Wire Wire Line
-	8175 4100 8300 4100
+Connection ~ 7500 4100
+Wire Wire Line
+	7500 4100 7600 4100
+Wire Wire Line
+	7500 4350 7600 4350
+Wire Wire Line
+	7500 4100 7500 4350
+Wire Wire Line
+	7400 4100 7500 4100
+Wire Wire Line
+	7000 4100 6900 4100
 Connection ~ 8175 4100
 Wire Wire Line
-	8175 3550 8175 3425
-Wire Wire Line
-	8175 3125 8175 3000
-Text GLabel 8300 4100 2    50   Output ~ 0
-IND_3
-Text Notes 8300 3450 0    50   ~ 0
-Yellow
+	7900 4100 8175 4100
 $EndSCHEMATC

Commit message: blah blah blah
Other:
- note added: "Sheet 2: Buttons"
Changed lines of the file:
@@
 Wire Wire Line
 	7900 4100 8175 4100
+Text Notes 9675 6975 2    200  ~ 40
+Sheet 2: Buttons
 $EndSCHEMATC

Commit message: Added values for buck components
Parts:
- gave numbers to parts that had none: 15
Changed lines of the file:
@@
 P 3975 3275
 AR Path="/5F4E4EE3" Ref="D?"  Part="1"
-AR Path="/5F4E3D8B/5F4E4EE3" Ref="D?"  Part="1"
-F 0 "D?" V 4014 3158 50  0000 R CNN
+AR Path="/5F4E3D8B/5F4E4EE3" Ref="D1"  Part="1"
+F 0 "D1" V 4014 3158 50  0000 R CNN
 F 1 "LED" V 3923 3158 50  0000 R CNN
 F 2 "" H 3975 3275 50  0001 C CNN
@@
 $EndComp
 $Comp
-L Device:R R?
+L Device:R R3
 U 1 1 5F566AF5
 P 3975 3700
-F 0 "R?" H 4045 3746 50  0000 L CNN
+F 0 "R3" H 4045 3746 50  0000 L CNN
 F 1 "10k" H 4045 3655 50  0000 L CNN
 F 2 "" V 3905 3700 50  0001 C CNN
@@
 $EndComp
 $Comp
-L Device:C C?
+L Device:C C1
 U 1 1 5F566E39
 P 3975 4400
-F 0 "C?" H 4090 4446 50  0000 L CNN
+F 0 "C1" H 4090 4446 50  0000 L CNN
 F 1 "0.1uF" H 4090 4355 50  0000 L CNN
 F 2 "" H 4013 4250 50  0001 C CNN
@@
 $EndComp
 $Comp
-L power:+3.3V #PWR?
+L power:+3.3V #PWR02
 U 1 1 5F567F50
 P 3975 3000
-F 0 "#PWR?" H 3975 2850 50  0001 C CNN
+F 0 "#PWR02" H 3975 2850 50  0001 C CNN
 F 1 "+3.3V" H 3990 3173 50  0000 C CNN
 F 2 "" H 3975 3000 50  0001 C CNN
@@
 $EndComp
 $Comp
-L power:GND #PWR?
+L power:GND #PWR03
 U 1 1 5F56A4E8
 P 3975 4650
-F 0 "#PWR?" H 3975 4400 50  0001 C CNN
+F 0 "#PWR03" H 3975 4400 50  0001 C CNN
 F 1 "GND" H 3980 4477 50  0000 C CNN
 F 2 "" H 3975 4650 50  0001 C CNN
@@
 P 6075 3275
 AR Path="/5F56DB99" Ref="D?"  Part="1"
-AR Path="/5F4E3D8B/5F56DB99" Ref="D?"  Part="1"
-F 0 "D?" V 6114 3158 50  0000 R CNN
+AR Path="/5F4E3D8B/5F56DB99" Ref="D2"  Part="1"
+F 0 "D2" V 6114 3158 50  0000 R CNN
 F 1 "LED" V 6023 3158 50  0000 R CNN
 F 2 "" H 6075 3275 50  0001 C CNN
@@
 $EndComp
 $Comp
-L Switch:SW_Push SW?
+L Switch:SW_Push SW2
 U 1 1 5F56DB9F
 P 5100 4100
-F 0 "SW?" H 5100 4385 50  0000 C CNN
+F 0 "SW2" H 5100 4385 50  0000 C CNN
 F 1 "SW_Push" H 5100 4294 50  0000 C CNN
 F 2 "" H 5100 4300 50  0001 C CNN
@@
 $EndComp
 $Comp
-L Device:R R?
+L Device:R R5
 U 1 1 5F56DBA5
 P 6075 3700
-F 0 "R?" H 6145 3746 50  0000 L CNN
+F 0 "R5" H 6145 3746 50  0000 L CNN
 F 1 "10k" H 6145 3655 50  0000 L CNN
 F 2 "" V 6005 3700 50  0001 C CNN
@@
 $EndComp
 $Comp
-L Device:C C?
+L Device:C C2
 U 1 1 5F56DBAB
 P 6075 4400
-F 0 "C?" H 6190 4446 50  0000 L CNN
+F 0 "C2" H 6190 4446 50  0000 L CNN
 F 1 "0.1uF" H 6190 4355 50  0000 L CNN
 F 2 "" H 6113 4250 50  0001 C CNN
@@
 $EndComp
 $Comp
-L power:GND #PWR?
+L power:GND #PWR04
 U 1 1 5F56DBB1
 P 4800 4200
-F 0 "#PWR?" H 4800 3950 50  0001 C CNN
+F 0 "#PWR04" H 4800 3950 50  0001 C CNN
 F 1 "GND" H 4805 4027 50  0000 C CNN
 F 2 "" H 4800 4200 50  0001 C CNN
@@
 $EndComp
 $Comp
-L power:+3.3V #PWR?
+L power:+3.3V #PWR05
 U 1 1 5F56DBB7
 P 6075 3000
-F 0 "#PWR?" H 6075 2850 50  0001 C CNN
+F 0 "#PWR05" H 6075 2850 50  0001 C CNN
 F 1 "+3.3V" H 6090 3173 50  0000 C CNN
 F 2 "" H 6075 3000 50  0001 C CNN
@@
 $EndComp
 $Comp
-L power:GND #PWR?
+L power:GND #PWR06
 U 1 1 5F56DBC3
 P 6075 4650
-F 0 "#PWR?" H 6075 4400 50  0001 C CNN
+F 0 "#PWR06" H 6075 4400 50  0001 C CNN
 F 1 "GND" H 6080 4477 50  0000 C CNN
 F 2 "" H 6075 4650 50  0001 C CNN
@@
 P 8175 3275
 AR Path="/5F5739F1" Ref="D?"  Part="1"
-AR Path="/5F4E3D8B/5F5739F1" Ref="D?"  Part="1"
-F 0 "D?" V 8214 3158 50  0000 R CNN
+AR Path="/5F4E3D8B/5F5739F1" Ref="D3"  Part="1"
+F 0 "D3" V 8214 3158 50  0000 R CNN
 F 1 "LED" V 8123 3158 50  0000 R CNN
 F 2 "" H 8175 3275 50  0001 C CNN
@@
 $EndComp
 $Comp
-L Device:R R?
+L Device:R R7
 U 1 1 5F5739FD
 P 8175 3700
-F 0 "R?" H 8245 3746 50  0000 L CNN
+F 0 "R7" H 8245 3746 50  0000 L CNN
 F 1 "10k" H 8245 3655 50  0000 L CNN
 F 2 "" V 8105 3700 50  0001 C CNN
@@
 $EndComp
 $Comp
-L Device:C C?
+L Device:C C3
 U 1 1 5F573A03
 P 8175 4400
-F 0 "C?" H 8290 4446 50  0000 L CNN
+F 0 "C3" H 8290 4446 50  0000 L CNN
 F 1 "0.1uF" H 8290 4355 50  0000 L CNN
 F 2 "" H 8213 4250 50  0001 C CNN
@@
 $EndComp
 $Comp
-L power:+3.3V #PWR?
+L power:+3.3V #PWR08
 U 1 1 5F573A0F
 P 8175 3000
-F 0 "#PWR?" H 8175 2850 50  0001 C CNN
+F 0 "#PWR08" H 8175 2850 50  0001 C CNN
 F 1 "+3.3V" H 8190 3173 50  0000 C CNN
 F 2 "" H 8175 3000 50  0001 C CNN
@@
 $EndComp
 $Comp
-L power:GND #PWR?
+L power:GND #PWR09
 U 1 1 5F573A1B
 P 8175 4650
-F 0 "#PWR?" H 8175 4400 50  0001 C CNN
+F 0 "#PWR09" H 8175 4400 50  0001 C CNN
 F 1 "GND" H 8180 4477 50  0000 C CNN
 F 2 "" H 8175 4650 50  0001 C CNN
@@
 	5800 4100 6075 4100
 $Comp
-L Device:R R?
+L Device:R R4
 U 1 1 5F56DBBD
 P 5650 4100
-F 0 "R?" V 5825 4050 50  0000 L CNN
+F 0 "R4" V 5825 4050 50  0000 L CNN
 F 1 "1k" V 5750 4075 50  0000 L CNN
 F 2 "" V 5580 4100 50  0001 C CNN
@@
 Connection ~ 3300 4100
 $Comp
-L Device:R R?
+L Device:R R2
 U 1 1 5F58E0DD
 P 3550 4100
-F 0 "R?" V 3725 4050 50  0000 L CNN
+F 0 "R2" V 3725 4050 50  0000 L CNN
 F 1 "1k" V 3650 4075 50  0000 L CNN
 F 2 "" V 3480 4100 50  0001 C CNN
@@
 	2700 4200 2700 4100
 $Comp
-L power:GND #PWR?
+L power:GND #PWR01
 U 1 1 5F58E0D5
 P 2700 4200
-F 0 "#PWR?" H 2700 3950 50  0001 C CNN
+F 0 "#PWR01" H 2700 3950 50  0001 C CNN
 F 1 "GND" H 2705 4027 50  0000 C CNN
 F 2 "" H 2700 4200 50  0001 C CNN
@@
 $EndComp
 $Comp
-L Switch:SW_Push SW?
+L Switch:SW_Push SW1
 U 1 1 5F58E0CF
 P 3000 4100
-F 0 "SW?" H 3000 4385 50  0000 C CNN
+F 0 "SW1" H 3000 4385 50  0000 C CNN
 F 1 "SW_Push" H 3000 4294 50  0000 C CNN
 F 2 "" H 3000 4300 50  0001 C CNN
@@
 	3700 4100 3975 4100
 $Comp
-L Switch:SW_Push SW?
+L Switch:SW_Push SW3
 U 1 1 5F595C41
 P 7200 4100
-F 0 "SW?" H 7200 4385 50  0000 C CNN
+F 0 "SW3" H 7200 4385 50  0000 C CNN
 F 1 "SW_Push" H 7200 4294 50  0000 C CNN
 F 2 "" H 7200 4300 50  0001 C CNN
@@
 $EndComp
 $Comp
-L power:GND #PWR?
+L power:GND #PWR07
 U 1 1 5F595C47
 P 6900 4200
-F 0 "#PWR?" H 6900 3950 50  0001 C CNN
+F 0 "#PWR07" H 6900 3950 50  0001 C CNN
 F 1 "GND" H 6905 4027 50  0000 C CNN
 F 2 "" H 6900 4200 50  0001 C CNN
@@
 IND_3
 $Comp
-L Device:R R?
+L Device:R R6
 U 1 1 5F595C4F
 P 7750 4100
-F 0 "R?" V 7925 4050 50  0000 L CNN
+F 0 "R6" V 7925 4050 50  0000 L CNN
 F 1 "1k" V 7850 4075 50  0000 L CNN
 F 2 "" V 7680 4100 50  0001 C CNN
