File: Hardware/_autosave-TrainingBoard2020.sch (KiCad schematic (older format))
At the start: 1 part

Commit message: updated things
Parts:
- removed unit 3 of Conn1
Connections:
- net labels removed: +12VA
- wire segments 4 -> 3
Changed lines of the file:
@@
 Wire Wire Line
 	1375 1975 2075 1975
-$Comp
-L MRDT_Connectors:AndersonPP Conn1
-U 3 1 5F60051F
-P 950 1100
-F 0 "Conn1" H 1158 1487 60  0000 C CNN
-F 1 "AndersonPP" H 1158 1381 60  0000 C CNN
-F 2 "" H 800 550 60  0001 C CNN
-F 3 "" H 800 550 60  0001 C CNN
-	3    950  1100
-	1    0    0    -1
-$EndComp
-Wire Wire Line
-	1350 1000 2050 1000
-Wire Wire Line
-	2050 1000 2050 850
-$Comp
-L power:+12VA #PWR010
-U 1 1 5F601FA2
-P 2050 850
-F 0 "#PWR010" H 2050 700 50  0001 C CNN
-F 1 "+12VA" H 2065 1023 50  0000 C CNN
-F 2 "" H 2050 850 50  0001 C CNN
-F 3 "" H 2050 850 50  0001 C CNN
-	1    2050 850
-	1    0    0    -1
-$EndComp
 $Sheet
 S 2275 925  1425 875
@@
 F1 "TrainingBoard01.sch" 50
 F2 "+12VL" I L 2275 1500 50
-F3 "+3.3V" O R 3700 1175 50
-F4 "+5.0V" O R 3700 1500 50
+F3 "+3.3V" O R 3700 1500 50
 $EndSheet
+Wire Wire Line
+	1375 1500 2275 1500
 $EndSCHEMATC
