File: Hardware/TrainingBoard2020/TrainingBoard01.sch (KiCad schematic (older format))
At the start: 13 parts, among them J1 Test_Point, J2 Test_Point, U1 LM2576D2TR4-3.3G

Commit message: Finished PCB layout
Parts:
- C1: footprint (none) -> Capacitor_SMD:C_Elec_5x5.4
- C2: footprint (none) -> Capacitor_SMD:C_Elec_8x5.4
- D1, D3: footprint (none) -> Diode_SMD:D_SOD-323_HandSoldering
- D2, D4: footprint (none) -> LED_SMD:LED_0603_1608Metric_Pad1.05x0.95mm_HandSolder
- FB1: footprint (none) -> Capacitor_SMD:C_0805_2012Metric_Pad1.15x1.40mm_HandSolder
- J1, J2: footprint (none) -> TestPoint:TestPoint_Pad_D2.5mm
- L1: footprint (none) -> Inductor_SMD:L_0603_1608Metric_Pad1.05x0.95mm_HandSolder
- R1, R2: footprint (none) -> Resistor_SMD:R_0603_1608Metric_Pad1.05x0.95mm_HandSolder
- U1: footprint (none) -> MRDT_Devices:LM2576; symbol MRDT_Devices:LM2576D2TR4-3.3G -> TrainingBoard2020-rescue:LM2576D2TR4-3.3G-MRDT_Devices
Connections:
- net Power_Input is gone; now on net +12V: D1.1 (K), FB1.2
Changed lines of the file:
@@
 Power_Input
 Wire Wire Line
-	2200 2550 2450 2550
+	2200 2550 2300 2550
 $Comp
 L Device:Ferrite_Bead FB1
@@
 F 0 "FB1" V 2476 2550 50  0000 C CNN
 F 1 "Ferrite_Bead" V 2567 2550 50  0000 C CNN
-F 2 "" V 2680 2550 50  0001 C CNN
+F 2 "Capacitor_SMD:C_0805_2012Metric_Pad1.15x1.40mm_HandSolder" V 2680 2550 50  0001 C CNN
 F 3 "~" H 2750 2550 50  0001 C CNN
 	1    2750 2550
@@
 F 0 "D1" V 2404 2930 50  0000 L CNN
 F 1 "D_Zener" V 2495 2930 50  0000 L CNN
-F 2 "" H 2450 2850 50  0001 C CNN
+F 2 "Diode_SMD:D_SOD-323_HandSoldering" H 2450 2850 50  0001 C CNN
 F 3 "~" H 2450 2850 50  0001 C CNN
 	1    2450 2850
@@
 F 0 "D2" H 3993 2295 50  0000 C CNN
 F 1 "LED" H 3993 2386 50  0000 C CNN
-F 2 "" H 4000 2550 50  0001 C CNN
+F 2 "LED_SMD:LED_0603_1608Metric_Pad1.05x0.95mm_HandSolder" H 4000 2550 50  0001 C CNN
 F 3 "~" H 4000 2550 50  0001 C CNN
 	1    4000 2550
@@
 F 0 "R1" V 4343 2550 50  0000 C CNN
 F 1 "1k" V 4434 2550 50  0000 C CNN
-F 2 "" V 4480 2550 50  0001 C CNN
+F 2 "Resistor_SMD:R_0603_1608Metric_Pad1.05x0.95mm_HandSolder" V 4480 2550 50  0001 C CNN
 F 3 "~" H 4550 2550 50  0001 C CNN
 	1    4550 2550
@@
 Green
 $Comp
-L MRDT_Devices:LM2576D2TR4-3.3G U1
+L TrainingBoard2020-rescue:LM2576D2TR4-3.3G-MRDT_Devices U1
 U 1 1 5F571CC8
 P 5850 4400
+AR Path="/5F571CC8" Ref="U1"  Part="1"
+AR Path="/5F56719A/5F571CC8" Ref="U1"  Part="1"
 F 0 "U1" H 5850 4825 50  0000 C CNN
 F 1 "LM2576D2TR4-3.3G" H 5850 4734 50  0000 C CNN
-F 2 "" H 5850 4850 50  0001 C CNN
+F 2 "MRDT_Devices:LM2576" H 5850 4850 50  0001 C CNN
 F 3 "https://www.mouser.com/datasheet/2/308/LM2576_D-1810688.pdf" H 5850 4850 50  0001 C CNN
 	1    5850 4400
@@
 F 0 "C1" V 6698 3950 50  0000 C CNN
 F 1 "100uF" V 6789 3950 50  0000 C CNN
-F 2 "" H 6988 3800 50  0001 C CNN
+F 2 "Capacitor_SMD:C_Elec_5x5.4" H 6988 3800 50  0001 C CNN
 F 3 "~" H 6950 3950 50  0001 C CNN
 	1    6950 3950
@@
 F 0 "D3" V 6654 4630 50  0000 L CNN
 F 1 "D_Zener" V 6745 4630 50  0000 L CNN
-F 2 "" H 6700 4550 50  0001 C CNN
+F 2 "Diode_SMD:D_SOD-323_HandSoldering" H 6700 4550 50  0001 C CNN
 F 3 "~" H 6700 4550 50  0001 C CNN
 	1    6700 4550
@@
 F 0 "L1" V 7290 4350 50  0000 C CNN
 F 1 "100mH" V 7199 4350 50  0000 C CNN
-F 2 "" H 7100 4350 50  0001 C CNN
+F 2 "Inductor_SMD:L_0603_1608Metric_Pad1.05x0.95mm_HandSolder" H 7100 4350 50  0001 C CNN
 F 3 "~" H 7100 4350 50  0001 C CNN
 	1    7100 4350
@@
 F 0 "C2" H 7450 4650 50  0000 C CNN
 F 1 "1000uF" H 7450 4550 50  0000 C CNN
-F 2 "" H 7738 4450 50  0001 C CNN
+F 2 "Capacitor_SMD:C_Elec_8x5.4" H 7738 4450 50  0001 C CNN
 F 3 "~" H 7700 4600 50  0001 C CNN
 	1    7700 4600
@@
 	7700 4750 7700 4850
 Wire Wire Line
-	8300 4350 8300 4100
+	8300 4350 8300 4150
 $Comp
 L power:+3.3V #PWR010
@@
 F 0 "R2" V 9043 4350 50  0000 C CNN
 F 1 "330" V 9134 4350 50  0000 C CNN
-F 2 "" V 9180 4350 50  0001 C CNN
+F 2 "Resistor_SMD:R_0603_1608Metric_Pad1.05x0.95mm_HandSolder" V 9180 4350 50  0001 C CNN
 F 3 "~" H 9250 4350 50  0001 C CNN
 	1    9250 4350
@@
 F 0 "J2" H 8300 4750 60  0000 L CNN
 F 1 "Test_Point" H 7950 4650 60  0000 L CNN
-F 2 "" H 8500 4550 60  0001 C CNN
+F 2 "TestPoint:TestPoint_Pad_D2.5mm" H 8500 4550 60  0001 C CNN
 F 3 "" H 8500 4550 60  0001 C CNN
 	1    8500 4600
@@
 F 0 "J1" H 3828 2845 60  0000 L CNN
 F 1 "Test_Point" H 3828 2739 60  0000 L CNN
-F 2 "" H 3750 2650 60  0001 C CNN
+F 2 "TestPoint:TestPoint_Pad_D2.5mm" H 3750 2650 60  0001 C CNN
 F 3 "" H 3750 2650 60  0001 C CNN
 	1    3750 2700
@@
 F 0 "D4" H 8693 4095 50  0000 C CNN
 F 1 "LED" H 8693 4186 50  0000 C CNN
-F 2 "" H 8700 4350 50  0001 C CNN
+F 2 "LED_SMD:LED_0603_1608Metric_Pad1.05x0.95mm_HandSolder" H 8700 4350 50  0001 C CNN
 F 3 "~" H 8700 4350 50  0001 C CNN
 	1    8700 4350
@@
 Text Notes 7600 3550 0    98   ~ 20
 3.3v Convertor
+Text HLabel 2150 2750 0    50   Input ~ 0
++12V
+Wire Wire Line
+	2150 2750 2300 2750
+Wire Wire Line
+	2300 2750 2300 2550
+Connection ~ 2300 2550
+Wire Wire Line
+	2300 2550 2450 2550
+Text HLabel 8000 3950 0    50   Input ~ 0
++3.3V
+Wire Wire Line
+	8000 3950 8150 3950
+Wire Wire Line
+	8150 3950 8150 4150
+Wire Wire Line
+	8150 4150 8300 4150
+Connection ~ 8300 4150
+Wire Wire Line
+	8300 4150 8300 4100
 $EndSCHEMATC
