File: Hardware/TrainingBoard2020/TrainingBoard02.sch (KiCad schematic (older format))
At the start: 15 parts, among them SW1 SW_Push, SW2 SW_Push, SW3 SW_Push

Commit message: Finished PCB layout
Parts:
- C3, C4, C5: footprint (none) -> Capacitor_SMD:C_0603_1608Metric_Pad1.05x0.95mm_HandSolder
- D5, D6, D7: footprint (none) -> LED_SMD:LED_0603_1608Metric_Pad1.05x0.95mm_HandSolder
- R3, R4, R5, R6, R7, R8: footprint (none) -> Resistor_SMD:R_0603_1608Metric_Pad1.05x0.95mm_HandSolder
- SW1, SW2, SW3: footprint (none) -> Button_Switch_SMD:SW_Push_1P1T_NO_6x6mm_H9.5mm
Changed lines of the file:
@@
 F 0 "SW1" H 3000 3985 50  0000 C CNN
 F 1 "SW_Push" H 3000 3894 50  0000 C CNN
-F 2 "" H 3000 3900 50  0001 C CNN
+F 2 "Button_Switch_SMD:SW_Push_1P1T_NO_6x6mm_H9.5mm" H 3000 3900 50  0001 C CNN
 F 3 "~" H 3000 3900 50  0001 C CNN
 	1    3000 3700
@@
 F 0 "D5" V 3789 2832 50  0000 R CNN
 F 1 "LED" V 3698 2832 50  0000 R CNN
-F 2 "" H 3750 2950 50  0001 C CNN
+F 2 "LED_SMD:LED_0603_1608Metric_Pad1.05x0.95mm_HandSolder" H 3750 2950 50  0001 C CNN
 F 3 "~" H 3750 2950 50  0001 C CNN
 	1    3750 2950
@@
 F 0 "R4" H 3820 3396 50  0000 L CNN
 F 1 "1k" H 3820 3305 50  0000 L CNN
-F 2 "" V 3680 3350 50  0001 C CNN
+F 2 "Resistor_SMD:R_0603_1608Metric_Pad1.05x0.95mm_HandSolder" V 3680 3350 50  0001 C CNN
 F 3 "~" H 3750 3350 50  0001 C CNN
 	1    3750 3350
@@
 F 0 "R3" V 3657 3700 50  0000 C CNN
 F 1 "1k" V 3566 3700 50  0000 C CNN
-F 2 "" V 3380 3700 50  0001 C CNN
+F 2 "Resistor_SMD:R_0603_1608Metric_Pad1.05x0.95mm_HandSolder" V 3380 3700 50  0001 C CNN
 F 3 "~" H 3450 3700 50  0001 C CNN
 	1    3450 3700
@@
 F 0 "C3" H 3865 4096 50  0000 L CNN
 F 1 "0.1uF" H 3865 4005 50  0000 L CNN
-F 2 "" H 3788 3900 50  0001 C CNN
+F 2 "Capacitor_SMD:C_0603_1608Metric_Pad1.05x0.95mm_HandSolder" H 3788 3900 50  0001 C CNN
 F 3 "~" H 3750 4050 50  0001 C CNN
 	1    3750 4050
@@
 F 0 "SW2" H 5250 3985 50  0000 C CNN
 F 1 "SW_Push" H 5250 3894 50  0000 C CNN
-F 2 "" H 5250 3900 50  0001 C CNN
+F 2 "Button_Switch_SMD:SW_Push_1P1T_NO_6x6mm_H9.5mm" H 5250 3900 50  0001 C CNN
 F 3 "~" H 5250 3900 50  0001 C CNN
 	1    5250 3700
@@
 F 0 "D6" V 6039 2832 50  0000 R CNN
 F 1 "LED" V 5948 2832 50  0000 R CNN
-F 2 "" H 6000 2950 50  0001 C CNN
+F 2 "LED_SMD:LED_0603_1608Metric_Pad1.05x0.95mm_HandSolder" H 6000 2950 50  0001 C CNN
 F 3 "~" H 6000 2950 50  0001 C CNN
 	1    6000 2950
@@
 F 0 "R6" H 6070 3396 50  0000 L CNN
 F 1 "1k" H 6070 3305 50  0000 L CNN
-F 2 "" V 5930 3350 50  0001 C CNN
+F 2 "Resistor_SMD:R_0603_1608Metric_Pad1.05x0.95mm_HandSolder" V 5930 3350 50  0001 C CNN
 F 3 "~" H 6000 3350 50  0001 C CNN
 	1    6000 3350
@@
 F 0 "R5" V 5907 3700 50  0000 C CNN
 F 1 "1k" V 5816 3700 50  0000 C CNN
-F 2 "" V 5630 3700 50  0001 C CNN
+F 2 "Resistor_SMD:R_0603_1608Metric_Pad1.05x0.95mm_HandSolder" V 5630 3700 50  0001 C CNN
 F 3 "~" H 5700 3700 50  0001 C CNN
 	1    5700 3700
@@
 F 0 "C4" H 6115 4096 50  0000 L CNN
 F 1 "0.1uF" H 6115 4005 50  0000 L CNN
-F 2 "" H 6038 3900 50  0001 C CNN
+F 2 "Capacitor_SMD:C_0603_1608Metric_Pad1.05x0.95mm_HandSolder" H 6038 3900 50  0001 C CNN
 F 3 "~" H 6000 4050 50  0001 C CNN
 	1    6000 4050
@@
 F 0 "SW3" H 7500 3985 50  0000 C CNN
 F 1 "SW_Push" H 7500 3894 50  0000 C CNN
-F 2 "" H 7500 3900 50  0001 C CNN
+F 2 "Button_Switch_SMD:SW_Push_1P1T_NO_6x6mm_H9.5mm" H 7500 3900 50  0001 C CNN
 F 3 "~" H 7500 3900 50  0001 C CNN
 	1    7500 3700
@@
 F 0 "D7" V 8289 2832 50  0000 R CNN
 F 1 "LED" V 8198 2832 50  0000 R CNN
-F 2 "" H 8250 2950 50  0001 C CNN
+F 2 "LED_SMD:LED_0603_1608Metric_Pad1.05x0.95mm_HandSolder" H 8250 2950 50  0001 C CNN
 F 3 "~" H 8250 2950 50  0001 C CNN
 	1    8250 2950
@@
 F 0 "R8" H 8320 3396 50  0000 L CNN
 F 1 "1k" H 8320 3305 50  0000 L CNN
-F 2 "" V 8180 3350 50  0001 C CNN
+F 2 "Resistor_SMD:R_0603_1608Metric_Pad1.05x0.95mm_HandSolder" V 8180 3350 50  0001 C CNN
 F 3 "~" H 8250 3350 50  0001 C CNN
 	1    8250 3350
@@
 F 0 "R7" V 8157 3700 50  0000 C CNN
 F 1 "1k" V 8066 3700 50  0000 C CNN
-F 2 "" V 7880 3700 50  0001 C CNN
+F 2 "Resistor_SMD:R_0603_1608Metric_Pad1.05x0.95mm_HandSolder" V 7880 3700 50  0001 C CNN
 F 3 "~" H 7950 3700 50  0001 C CNN
 	1    7950 3700
@@
 F 0 "C5" H 8365 4096 50  0000 L CNN
 F 1 "0.1uF" H 8365 4005 50  0000 L CNN
-F 2 "" H 8288 3900 50  0001 C CNN
+F 2 "Capacitor_SMD:C_0603_1608Metric_Pad1.05x0.95mm_HandSolder" H 8288 3900 50  0001 C CNN
 F 3 "~" H 8250 4050 50  0001 C CNN
 	1    8250 4050
