File: Hardware/TrainingBoard2020/TraininbBoard01.sch (KiCad schematic (older format))
At the start: 13 parts

Commit message: Didn't save before committing
Parts:
- gave numbers to parts that had none: 13
Changed lines of the file:
@@
 	2900 1900 3500 1900
 $Comp
-L Device:Ferrite_Bead FB?
+L Device:Ferrite_Bead FB1
 U 1 1 5F685143
 P 4150 1900
-F 0 "FB?" V 3876 1900 50  0000 C CNN
+F 0 "FB1" V 3876 1900 50  0000 C CNN
 F 1 "Ferrite_Bead" V 3967 1900 50  0000 C CNN
 F 2 "" V 4080 1900 50  0001 C CNN
@@
 $EndComp
 $Comp
-L Device:D_Zener D?
+L Device:D_Zener D1
 U 1 1 5F685BAD
 P 3500 2050
-F 0 "D?" V 3454 2130 50  0000 L CNN
+F 0 "D1" V 3454 2130 50  0000 L CNN
 F 1 "D_Zener" V 3545 2130 50  0000 L CNN
 F 2 "" H 3500 2050 50  0001 C CNN
@@
 	3500 2200 3500 2500
 $Comp
-L power:GND #PWR?
+L power:GND #PWR01
 U 1 1 5F686F50
 P 3500 2500
-F 0 "#PWR?" H 3500 2250 50  0001 C CNN
+F 0 "#PWR01" H 3500 2250 50  0001 C CNN
 F 1 "GND" H 3505 2327 50  0000 C CNN
 F 2 "" H 3500 2500 50  0001 C CNN
@@
 	4950 1900 4950 1600
 $Comp
-L power:+12V #PWR?
+L power:+12V #PWR02
 U 1 1 5F6875BA
 P 4950 1600
-F 0 "#PWR?" H 4950 1450 50  0001 C CNN
+F 0 "#PWR02" H 4950 1450 50  0001 C CNN
 F 1 "+12V" H 4965 1773 50  0000 C CNN
 F 2 "" H 4950 1600 50  0001 C CNN
@@
 Connection ~ 4950 1900
 $Comp
-L Device:LED D?
+L Device:LED D2
 U 1 1 5F687E2D
 P 5550 1900
-F 0 "D?" H 5543 1645 50  0000 C CNN
+F 0 "D2" H 5543 1645 50  0000 C CNN
 F 1 "LED" H 5543 1736 50  0000 C CNN
 F 2 "" H 5550 1900 50  0001 C CNN
@@
 $EndComp
 $Comp
-L Device:R R?
+L Device:R R1
 U 1 1 5F688767
 P 6100 1900
-F 0 "R?" V 5893 1900 50  0000 C CNN
+F 0 "R1" V 5893 1900 50  0000 C CNN
 F 1 "1k" V 5984 1900 50  0000 C CNN
 F 2 "" V 6030 1900 50  0001 C CNN
@@
 $EndComp
 $Comp
-L power:GND #PWR?
+L power:GND #PWR04
 U 1 1 5F689446
 P 6500 2150
-F 0 "#PWR?" H 6500 1900 50  0001 C CNN
+F 0 "#PWR04" H 6500 1900 50  0001 C CNN
 F 1 "GND" H 6505 1977 50  0000 C CNN
 F 2 "" H 6500 2150 50  0001 C CNN
@@
 Green
 $Comp
-L power:GND #PWR?
+L power:GND #PWR03
 U 1 1 5F68B343
 P 5400 3950
-F 0 "#PWR?" H 5400 3700 50  0001 C CNN
+F 0 "#PWR03" H 5400 3700 50  0001 C CNN
 F 1 "GND" H 5405 3777 50  0000 C CNN
 F 2 "" H 5400 3950 50  0001 C CNN
@@
 	5400 3650 5400 3800
 $Comp
-L MRDT_Devices:LM2576D2TR4 U?
+L MRDT_Devices:LM2576D2TR4 U1
 U 1 1 5F689B52
 P 6500 3700
-F 0 "U?" H 6500 4125 50  0000 C CNN
+F 0 "U1" H 6500 4125 50  0000 C CNN
 F 1 "LM2576D2TR4" H 6500 4034 50  0000 C CNN
 F 2 "" H 6500 4150 50  0001 C CNN
@@
 	5400 3950 5400 4000
 $Comp
-L power:+12V #PWR?
+L power:+12V #PWR05
 U 1 1 5F68EBB6
 P 7150 3150
-F 0 "#PWR?" H 7150 3000 50  0001 C CNN
+F 0 "#PWR05" H 7150 3000 50  0001 C CNN
 F 1 "+12V" H 7165 3323 50  0000 C CNN
 F 2 "" H 7150 3150 50  0001 C CNN
@@
 $EndComp
 $Comp
-L Device:C C?
+L Device:C C1
 U 1 1 5F68ED1D
 P 7350 3300
-F 0 "C?" V 7098 3300 50  0000 C CNN
+F 0 "C1" V 7098 3300 50  0000 C CNN
 F 1 "100uF" V 7189 3300 50  0000 C CNN
 F 2 "" H 7388 3150 50  0001 C CNN
@@
 $EndComp
 $Comp
-L power:GND #PWR?
+L power:GND #PWR07
 U 1 1 5F68F84F
 P 7900 3300
-F 0 "#PWR?" H 7900 3050 50  0001 C CNN
+F 0 "#PWR07" H 7900 3050 50  0001 C CNN
 F 1 "GND" H 7905 3127 50  0000 C CNN
 F 2 "" H 7900 3300 50  0001 C CNN
@@
 	7900 3300 7900 3350
 $Comp
-L Device:D_Zener D?
+L Device:D_Zener D3
 U 1 1 5F691AD7
 P 7250 3850
-F 0 "D?" V 7204 3930 50  0000 L CNN
+F 0 "D3" V 7204 3930 50  0000 L CNN
 F 1 "D_Zener" V 7295 3930 50  0000 L CNN
 F 2 "" H 7250 3850 50  0001 C CNN
@@
 	7250 3650 7400 3650
 $Comp
-L Device:L L?
+L Device:L L1
 U 1 1 5F692502
 P 7550 3650
-F 0 "L?" V 7369 3650 50  0000 C CNN
+F 0 "L1" V 7369 3650 50  0000 C CNN
 F 1 "100uH" V 7460 3650 50  0000 C CNN
 F 2 "" H 7550 3650 50  0001 C CNN
@@
 Connection ~ 7900 3300
 $Comp
-L power:GND #PWR?
+L power:GND #PWR06
 U 1 1 5F69676C
 P 7250 4100
-F 0 "#PWR?" H 7250 3850 50  0001 C CNN
+F 0 "#PWR06" H 7250 3850 50  0001 C CNN
 F 1 "GND" H 7255 3927 50  0000 C CNN
 F 2 "" H 7250 4100 50  0001 C CNN
@@
 Connection ~ 7750 3650
 $Comp
-L Device:C C?
+L Device:C C2
 U 1 1 5F697ED0
 P 8100 3900
-F 0 "C?" H 8215 3946 50  0000 L CNN
+F 0 "C2" H 8215 3946 50  0000 L CNN
 F 1 "1000uF" H 8215 3855 50  0000 L CNN
 F 2 "" H 8138 3750 50  0001 C CNN
@@
 Connection ~ 8100 3650
 $Comp
-L power:GND #PWR?
+L power:GND #PWR08
 U 1 1 5F699E4F
 P 8100 4200
-F 0 "#PWR?" H 8100 3950 50  0001 C CNN
+F 0 "#PWR08" H 8100 3950 50  0001 C CNN
 F 1 "GND" H 8105 4027 50  0000 C CNN
 F 2 "" H 8100 4200 50  0001 C CNN
@@
 	8100 3650 8550 3650
 $Comp
-L power:+3.3V #PWR?
+L power:+3.3V #PWR09
 U 1 1 5F69AE49
 P 8550 3300
-F 0 "#PWR?" H 8550 3150 50  0001 C CNN
+F 0 "#PWR09" H 8550 3150 50  0001 C CNN
 F 1 "+3.3V" H 8565 3473 50  0000 C CNN
 F 2 "" H 8550 3300 50  0001 C CNN
@@
 	8550 3650 8850 3650
 $Comp
-L Device:LED D?
+L Device:LED D4
 U 1 1 5F69DC2F
 P 9150 3650
-F 0 "D?" H 9143 3395 50  0000 C CNN
+F 0 "D4" H 9143 3395 50  0000 C CNN
 F 1 "LED" H 9143 3486 50  0000 C CNN
 F 2 "" H 9150 3650 50  0001 C CNN
@@
 $EndComp
 $Comp
-L Device:R R?
+L Device:R R2
 U 1 1 5F69DC35
 P 9700 3650
-F 0 "R?" V 9493 3650 50  0000 C CNN
+F 0 "R2" V 9493 3650 50  0000 C CNN
 F 1 "330" V 9584 3650 50  0000 C CNN
 F 2 "" V 9630 3650 50  0001 C CNN
@@
 $EndComp
 $Comp
-L power:GND #PWR?
+L power:GND #PWR010
 U 1 1 5F69DC3B
 P 10100 3900
-F 0 "#PWR?" H 10100 3650 50  0001 C CNN
+F 0 "#PWR010" H 10100 3650 50  0001 C CNN
 F 1 "GND" H 10105 3727 50  0000 C CNN
 F 2 "" H 10100 3900 50  0001 C CNN
@@
 Green
 $Comp
-L MRDT_Connectors:Test_Point J?
+L MRDT_Connectors:Test_Point J2
 U 1 1 5F69E5AD
 P 8850 3850
-F 0 "J?" H 8772 3889 60  0000 R CNN
+F 0 "J2" H 8772 3889 60  0000 R CNN
 F 1 "Test_Point" H 8772 3995 60  0000 R CNN
 F 2 "" H 8850 3800 60  0001 C CNN
@@
 	8850 3650 9000 3650
 $Comp
-L MRDT_Connectors:Test_Point J?
+L MRDT_Connectors:Test_Point J1
 U 1 1 5F6A7562
 P 4550 2100
-F 0 "J?" H 4472 2139 60  0000 R CNN
+F 0 "J1" H 4472 2139 60  0000 R CNN
 F 1 "Test_Point" H 4472 2245 60  0000 R CNN
 F 2 "" H 4550 2050 60  0001 C CNN
