File: Hardware/TrainingBoard2020/TraininbBoard02.sch (KiCad schematic (older format))
At the start: 15 parts

Commit message: Didn't save before committing
Parts:
- gave numbers to parts that had none: 15
Connections:
- net labels added: Ind_2, Ind_3
- wire segments 24 -> 28
Other:
- moved on the sheet: C4, D6, R5, R6, SW2
Changed lines of the file:
@@
 Sheet 02 Buttons\n
 $Comp
-L Switch:SW_Push SW?
+L Switch:SW_Push SW1
 U 1 1 5F6A8512
 P 1500 3350
-F 0 "SW?" H 1500 3635 50  0000 C CNN
+F 0 "SW1" H 1500 3635 50  0000 C CNN
 F 1 "SW_Push" H 1500 3544 50  0000 C CNN
 F 2 "" H 1500 3550 50  0001 C CNN
@@
 	1300 3350 950  3350
 $Comp
-L power:+3.3V #PWR?
+L power:+3.3V #PWR012
 U 1 1 5F6A8F03
 P 2550 2400
-F 0 "#PWR?" H 2550 2250 50  0001 C CNN
+F 0 "#PWR012" H 2550 2250 50  0001 C CNN
 F 1 "+3.3V" H 2565 2573 50  0000 C CNN
 F 2 "" H 2550 2400 50  0001 C CNN
@@
 $EndComp
 $Comp
-L Device:LED D?
+L Device:LED D5
 U 1 1 5F6A941B
 P 2550 2600
-F 0 "D?" V 2589 2482 50  0000 R CNN
+F 0 "D5" V 2589 2482 50  0000 R CNN
 F 1 "LED" V 2498 2482 50  0000 R CNN
 F 2 "" H 2550 2600 50  0001 C CNN
@@
 $EndComp
 $Comp
-L Device:R R?
+L Device:R R4
 U 1 1 5F6AA38F
 P 2550 3050
-F 0 "R?" H 2620 3096 50  0000 L CNN
+F 0 "R4" H 2620 3096 50  0000 L CNN
 F 1 "1k" H 2620 3005 50  0000 L CNN
 F 2 "" V 2480 3050 50  0001 C CNN
@@
 $EndComp
 $Comp
-L Device:R R?
+L Device:R R3
 U 1 1 5F6AADDC
 P 2350 3350
-F 0 "R?" V 2557 3350 50  0000 C CNN
+F 0 "R3" V 2557 3350 50  0000 C CNN
 F 1 "1k" V 2466 3350 50  0000 C CNN
 F 2 "" V 2280 3350 50  0001 C CNN
@@
 $EndComp
 $Comp
-L Device:C C?
+L Device:C C3
 U 1 1 5F6AB3DD
 P 2550 3650
-F 0 "C?" H 2665 3696 50  0000 L CNN
+F 0 "C3" H 2665 3696 50  0000 L CNN
 F 1 "0.1uF" H 2665 3605 50  0000 L CNN
 F 2 "" H 2588 3500 50  0001 C CNN
@@
 	2550 2750 2550 2900
 Wire Wire Line
-	2550 3200 2550 3350
+	2550 3200 2550 3250
 Wire Wire Line
 	2500 3350 2550 3350
@@
 	2200 3350 1700 3350
 $Comp
-L power:GND #PWR?
+L power:GND #PWR011
 U 1 1 5F6AC7F3
 P 950 3350
-F 0 "#PWR?" H 950 3100 50  0001 C CNN
+F 0 "#PWR011" H 950 3100 50  0001 C CNN
 F 1 "GND" H 955 3177 50  0000 C CNN
 F 2 "" H 950 3350 50  0001 C CNN
@@
 $EndComp
 $Comp
-L power:GND #PWR?
+L power:GND #PWR013
 U 1 1 5F6ACE43
 P 2550 3950
-F 0 "#PWR?" H 2550 3700 50  0001 C CNN
+F 0 "#PWR013" H 2550 3700 50  0001 C CNN
 F 1 "GND" H 2555 3777 50  0000 C CNN
 F 2 "" H 2550 3950 50  0001 C CNN
@@
 blue
 $Comp
-L Switch:SW_Push SW?
+L Switch:SW_Push SW2
 U 1 1 5F6B2D01
-P 3650 3350
-F 0 "SW?" H 3650 3635 50  0000 C CNN
-F 1 "SW_Push" H 3650 3544 50  0000 C CNN
-F 2 "" H 3650 3550 50  0001 C CNN
-F 3 "~" H 3650 3550 50  0001 C CNN
-	1    3650 3350
-	1    0    0    -1
-$EndComp
-Wire Wire Line
-	3450 3350 3100 3350
-$Comp
-L power:+3.3V #PWR?
+P 3950 3350
+F 0 "SW2" H 3950 3635 50  0000 C CNN
+F 1 "SW_Push" H 3950 3544 50  0000 C CNN
+F 2 "" H 3950 3550 50  0001 C CNN
+F 3 "~" H 3950 3550 50  0001 C CNN
+	1    3950 3350
+	1    0    0    -1
+$EndComp
+Wire Wire Line
+	3750 3350 3400 3350
+$Comp
+L power:+3.3V #PWR015
 U 1 1 5F6B2D08
-P 4700 2400
-F 0 "#PWR?" H 4700 2250 50  0001 C CNN
-F 1 "+3.3V" H 4715 2573 50  0000 C CNN
-F 2 "" H 4700 2400 50  0001 C CNN
-F 3 "" H 4700 2400 50  0001 C CNN
-	1    4700 2400
-	1    0    0    -1
-$EndComp
-$Comp
-L Device:LED D?
+P 5000 2400
+F 0 "#PWR015" H 5000 2250 50  0001 C CNN
+F 1 "+3.3V" H 5015 2573 50  0000 C CNN
+F 2 "" H 5000 2400 50  0001 C CNN
+F 3 "" H 5000 2400 50  0001 C CNN
+	1    5000 2400
+	1    0    0    -1
+$EndComp
+$Comp
+L Device:LED D6
 U 1 1 5F6B2D0E
-P 4700 2600
-F 0 "D?" V 4739 2482 50  0000 R CNN
-F 1 "LED" V 4648 2482 50  0000 R CNN
-F 2 "" H 4700 2600 50  0001 C CNN
-F 3 "~" H 4700 2600 50  0001 C CNN
-	1    4700 2600
-	0    -1   -1   0
-$EndComp
-$Comp
-L Device:R R?
+P 5000 2600
+F 0 "D6" V 5039 2482 50  0000 R CNN
+F 1 "LED" V 4948 2482 50  0000 R CNN
+F 2 "" H 5000 2600 50  0001 C CNN
+F 3 "~" H 5000 2600 50  0001 C CNN
+	1    5000 2600
+	0    -1   -1   0
+$EndComp
+$Comp
+L Device:R R6
 U 1 1 5F6B2D14
-P 4700 3050
-F 0 "R?" H 4770 3096 50  0000 L CNN
-F 1 "1k" H 4770 3005 50  0000 L CNN
-F 2 "" V 4630 3050 50  0001 C CNN
-F 3 "~" H 4700 3050 50  0001 C CNN
-	1    4700 3050
-	1    0    0    -1
-$EndComp
-$Comp
-L Device:R R?
+P 5000 3050
+F 0 "R6" H 5070 3096 50  0000 L CNN
+F 1 "1k" H 5070 3005 50  0000 L CNN
+F 2 "" V 4930 3050 50  0001 C CNN
+F 3 "~" H 5000 3050 50  0001 C CNN
+	1    5000 3050
+	1    0    0    -1
+$EndComp
+$Comp
+L Device:R R5
 U 1 1 5F6B2D1A
-P 4500 3350
-F 0 "R?" V 4707 3350 50  0000 C CNN
-F 1 "1k" V 4616 3350 50  0000 C CNN
-F 2 "" V 4430 3350 50  0001 C CNN
-F 3 "~" H 4500 3350 50  0001 C CNN
-	1    4500 3350
-	0    -1   -1   0
-$EndComp
-$Comp
-L Device:C C?
+P 4800 3350
+F 0 "R5" V 5007 3350 50  0000 C CNN
+F 1 "1k" V 4916 3350 50  0000 C CNN
+F 2 "" V 4730 3350 50  0001 C CNN
+F 3 "~" H 4800 3350 50  0001 C CNN
+	1    4800 3350
+	0    -1   -1   0
+$EndComp
+$Comp
+L Device:C C4
 U 1 1 5F6B2D20
-P 4700 3650
-F 0 "C?" H 4815 3696 50  0000 L CNN
-F 1 "0.1uF" H 4815 3605 50  0000 L CNN
-F 2 "" H 4738 3500 50  0001 C CNN
-F 3 "~" H 4700 3650 50  0001 C CNN
-	1    4700 3650
-	1    0    0    -1
-$EndComp
-Wire Wire Line
-	4700 2400 4700 2450
-Wire Wire Line
-	4700 2750 4700 2900
-Wire Wire Line
-	4700 3200 4700 3350
-Wire Wire Line
-	4650 3350 4700 3350
-Connection ~ 4700 3350
-Wire Wire Line
-	4700 3350 4700 3500
-Wire Wire Line
-	4350 3350 3850 3350
-$Comp
-L power:GND #PWR?
+P 5000 3650
+F 0 "C4" H 5115 3696 50  0000 L CNN
+F 1 "0.1uF" H 5115 3605 50  0000 L CNN
+F 2 "" H 5038 3500 50  0001 C CNN
+F 3 "~" H 5000 3650 50  0001 C CNN
+	1    5000 3650
+	1    0    0    -1
+$EndComp
+Wire Wire Line
+	5000 2400 5000 2450
+Wire Wire Line
+	5000 2750 5000 2900
+Wire Wire Line
+	5000 3200 5000 3350
+Wire Wire Line
+	4950 3350 5000 3350
+Connection ~ 5000 3350
+Wire Wire Line
+	5000 3350 5000 3500
+Wire Wire Line
+	4650 3350 4150 3350
+$Comp
+L power:GND #PWR014
 U 1 1 5F6B2D2D
-P 3100 3350
-F 0 "#PWR?" H 3100 3100 50  0001 C CNN
-F 1 "GND" H 3105 3177 50  0000 C CNN
-F 2 "" H 3100 3350 50  0001 C CNN
-F 3 "" H 3100 3350 50  0001 C CNN
-	1    3100 3350
-	1    0    0    -1
-$EndComp
-$Comp
-L power:GND #PWR?
+P 3400 3350
+F 0 "#PWR014" H 3400 3100 50  0001 C CNN
+F 1 "GND" H 3405 3177 50  0000 C CNN
+F 2 "" H 3400 3350 50  0001 C CNN
+F 3 "" H 3400 3350 50  0001 C CNN
+	1    3400 3350
+	1    0    0    -1
+$EndComp
+$Comp
+L power:GND #PWR016
 U 1 1 5F6B2D33
-P 4700 3950
-F 0 "#PWR?" H 4700 3700 50  0001 C CNN
-F 1 "GND" H 4705 3777 50  0000 C CNN
-F 2 "" H 4700 3950 50  0001 C CNN
-F 3 "" H 4700 3950 50  0001 C CNN
-	1    4700 3950
-	1    0    0    -1
-$EndComp
-Wire Wire Line
-	4700 3800 4700 3950
-Text Notes 5000 2650 0    79   ~ 0
+P 5000 3950
+F 0 "#PWR016" H 5000 3700 50  0001 C CNN
+F 1 "GND" H 5005 3777 50  0000 C CNN
+F 2 "" H 5000 3950 50  0001 C CNN
+F 3 "" H 5000 3950 50  0001 C CNN
+	1    5000 3950
+	1    0    0    -1
+$EndComp
+Wire Wire Line
+	5000 3800 5000 3950
+Text Notes 5300 2650 0    79   ~ 0
 blue
 $Comp
-L Switch:SW_Push SW?
+L Switch:SW_Push SW3
 U 1 1 5F6B8D6B
 P 6600 3350
-F 0 "SW?" H 6600 3635 50  0000 C CNN
+F 0 "SW3" H 6600 3635 50  0000 C CNN
 F 1 "SW_Push" H 6600 3544 50  0000 C CNN
 F 2 "" H 6600 3550 50  0001 C CNN
@@
 	6400 3350 6050 3350
 $Comp
-L power:+3.3V #PWR?
+L power:+3.3V #PWR018
 U 1 1 5F6B8D72
 P 7650 2400
-F 0 "#PWR?" H 7650 2250 50  0001 C CNN
+F 0 "#PWR018" H 7650 2250 50  0001 C CNN
 F 1 "+3.3V" H 7665 2573 50  0000 C CNN
 F 2 "" H 7650 2400 50  0001 C CNN
@@
 $EndComp
 $Comp
-L Device:LED D?
+L Device:LED D7
 U 1 1 5F6B8D78
 P 7650 2600
-F 0 "D?" V 7689 2482 50  0000 R CNN
+F 0 "D7" V 7689 2482 50  0000 R CNN
 F 1 "LED" V 7598 2482 50  0000 R CNN
 F 2 "" H 7650 2600 50  0001 C CNN
@@
 $EndComp
 $Comp
-L Device:R R?
+L Device:R R8
 U 1 1 5F6B8D7E
 P 7650 3050
-F 0 "R?" H 7720 3096 50  0000 L CNN
+F 0 "R8" H 7720 3096 50  0000 L CNN
 F 1 "1k" H 7720 3005 50  0000 L CNN
 F 2 "" V 7580 3050 50  0001 C CNN
@@
 $EndComp
 $Comp
-L Device:R R?
+L Device:R R7
 U 1 1 5F6B8D84
 P 7450 3350
-F 0 "R?" V 7657 3350 50  0000 C CNN
+F 0 "R7" V 7657 3350 50  0000 C CNN
 F 1 "1k" V 7566 3350 50  0000 C CNN
 F 2 "" V 7380 3350 50  0001 C CNN
@@
 $EndComp
 $Comp
-L Device:C C?
+L Device:C C5
 U 1 1 5F6B8D8A
 P 7650 3650
-F 0 "C?" H 7765 3696 50  0000 L CNN
+F 0 "C5" H 7765 3696 50  0000 L CNN
 F 1 "0.1uF" H 7765 3605 50  0000 L CNN
 F 2 "" H 7688 3500 50  0001 C CNN
@@
 	7300 3350 6800 3350
 $Comp
-L power:GND #PWR?
+L power:GND #PWR017
 U 1 1 5F6B8D97
 P 6050 3350
-F 0 "#PWR?" H 6050 3100 50  0001 C CNN
+F 0 "#PWR017" H 6050 3100 50  0001 C CNN
 F 1 "GND" H 6055 3177 50  0000 C CNN
 F 2 "" H 6050 3350 50  0001 C CNN
@@
 $EndComp
 $Comp
-L power:GND #PWR?
+L power:GND #PWR019
 U 1 1 5F6B8D9D
 P 7650 3950
-F 0 "#PWR?" H 7650 3700 50  0001 C CNN
+F 0 "#PWR019" H 7650 3700 50  0001 C CNN
 F 1 "GND" H 7655 3777 50  0000 C CNN
 F 2 "" H 7650 3950 50  0001 C CNN
@@
 Text Notes 7950 2650 0    79   ~ 0
 blue
-Text GLabel 3000 3950 2    79   Input ~ 0
+Text GLabel 2700 3250 2    79   Input ~ 0
 Ind_1
+Wire Wire Line
+	2700 3250 2550 3250
+Connection ~ 2550 3250
+Wire Wire Line
+	2550 3250 2550 3350
+Text GLabel 5150 3250 2    79   Input ~ 0
+Ind_2
+Wire Wire Line
+	5150 3250 5000 3250
+Text GLabel 7800 3250 2    79   Input ~ 0
+Ind_3
+Wire Wire Line
+	7800 3250 7650 3250
 $EndSCHEMATC
